Commit message: learning ROS

File: description/robot.urdf.xacro (robot description, xacro)
@@ -1,6 +1,5 @@
 <?xml version="1.0"?>
 <robot xmlns:xacro="http://www.ros.org/wiki/xacro"  name="robot">
-    <!-- Example link -->
-    <link name="base_link"></link>
+    <xacro:include filename="robot.core.xacro" />
 </robot>
 <!-- soon update -->
